File: USB_Audio_Interface.brd (EAGLE design)
At the start: 64.5 x 39 mm, 59 parts, among them IC1 PCM2904DB, IC2 OPA2353, IC3 AZ1117CH-ADJTRG1, J3 629722000214, Q1 12MHz

Commit message: Updated tValue positions for easy population
Parts:
- D1: value 5Vdc -> 82400102 5V
- D3: value 5Vdc -> 824022 5V

Commit message: Added population plan
Parts:
- L1: value 600Ohm@100 MHz -> 742792651
Changed lines of the file:
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@@
 <drawing>
 <settings>
-<setting alwaysvectorfont="yes"/>
+<setting alwaysvectorfont="no"/>
 <setting verticaltext="up"/>
 </settings>
@@
 <attribute name="VBR" value="6V" x="17.5" y="33" size="1" layer="27" rot="R270" display="off"/>
 </element>
-<element name="L1" library="Wurth_EMC Components_WE-CBF" library_urn="urn:adsk.eagle:library:14283147" package="WE-CBF_0603_W2.6" package3d_urn="urn:adsk.eagle:package:7784395/7" value="600Ohm@100 MHz" x="10.5" y="15.5" smashed="yes">
+<element name="L1" library="Wurth_EMC Components_WE-CBF" library_urn="urn:adsk.eagle:library:14283147" package="WE-CBF_0603_W2.6" package3d_urn="urn:adsk.eagle:package:7784395/7" value="742792651" x="10.5" y="15.5" smashed="yes">
 <attribute name="DATASHEET-URL" value="https://www.we-online.com/redexpert/spec/742792651?ae" x="10.5" y="15.5" size="1" layer="27" display="off"/>
 <attribute name="IR2" value="1000mA" x="10.5" y="15.5" size="1" layer="27" display="off"/>
