File: USB_Audio_Interface.sch (EAGLE design)
At the start: 59 parts, among them IC1 PCM2904DB, IC2 OPA2353, IC3 AZ1117CH-ADJTRG1, J3 629722000214, Q1 12MHz

Commit message: * Cleaned schematic a bit, exported new PDF * Cleaned up the PCB, USB has now its own netclass, updated GERBER * Updated image of PCB * Updated readme
Connections:
- net N$18 renamed !SSPND
Other:
- note added: "Electrolytics: Nichicon UCM1H100MCL6GS 12MHz Crystal: ECS-120-18-5P Case: Hammond 1455D601 Cinch/RCA connectors: BPJF02AUX BPJR04AUX"
- note added: "Inputs to GND"
- note added: "Left Antialiasing amp"
- note added: "Right Antialiasing amp"
- note added: "SJ1...4: Close 1-2 for Line Out Close 2-3 for Line In"
- note added: "To RCA connectors"
- note added: "https://github.com/SebiR/USB_Audio_Interface"
- note removed: "BPJF02AUX BPJR04AUX"
- note removed: "Case: 1455D601BK https://www.reichelt.de/profilgehaeuse-1455-d-60-x-45-x-25-mm-klar-1455d601-p221345.html?search=1455D"
- note removed: "ECS-120-18-5P"
- note removed: "Electrolytics: Nichicon UCM1H100MCL6GS"
- note removed: "Left channel pre-amp"
- note removed: "Right channel pre-amp"
- moved on the sheet: C10, C13, C20, C9, D2, D3, Q1, R11, R12, R13, R14, R17

Commit message: Updated tValue positions for easy population
Parts:
- D1: value 5Vdc -> 82400102 5V
- D3: value 5Vdc -> 824022 5V
Changed lines of the file:
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@@
 <part name="R18" library="rcl" library_urn="urn:adsk.eagle:library:334" deviceset="R-EU_" device="R0603" package3d_urn="urn:adsk.eagle:package:23555/3" value="330R"/>
 <part name="GND29" library="supply1" deviceset="GND" device=""/>
-<part name="D1" library="Wurth_EMC Components_WE-TVS" library_urn="urn:adsk.eagle:library:14282971" deviceset="WE-TVS-HS_SOT23-6L_82400102" device="" package3d_urn="urn:adsk.eagle:package:12152378/5" value="5Vdc"/>
+<part name="D1" library="Wurth_EMC Components_WE-TVS" library_urn="urn:adsk.eagle:library:14282971" deviceset="WE-TVS-HS_SOT23-6L_82400102" device="" package3d_urn="urn:adsk.eagle:package:12152378/5" value="82400102 5V"/>
 <part name="P+5" library="supply1" library_urn="urn:adsk.eagle:library:371" deviceset="+5V" device=""/>
 <part name="GND30" library="supply1" library_urn="urn:adsk.eagle:library:371" deviceset="GND" device=""/>
@@
 <part name="PAD2" library="wirepad" library_urn="urn:adsk.eagle:library:412" deviceset="2,15/1,0" device="" package3d_urn="urn:adsk.eagle:package:30831/1"/>
 <part name="PAD3" library="wirepad" library_urn="urn:adsk.eagle:library:412" deviceset="2,15/1,0" device="" package3d_urn="urn:adsk.eagle:package:30831/1"/>
-<part name="D3" library="Wurth_EMC Components_WE-TVS" library_urn="urn:adsk.eagle:library:14282971" deviceset="WE-TVS_SOT23-3L_824022" device="" package3d_urn="urn:adsk.eagle:package:12152380/4" value="5Vdc"/>
+<part name="D3" library="Wurth_EMC Components_WE-TVS" library_urn="urn:adsk.eagle:library:14282971" deviceset="WE-TVS_SOT23-3L_824022" device="" package3d_urn="urn:adsk.eagle:package:12152380/4" value="824022 5V"/>
 <part name="GND31" library="supply1" library_urn="urn:adsk.eagle:library:371" deviceset="GND" device=""/>
 <part name="SJ1" library="jumper" library_urn="urn:adsk.eagle:library:252" deviceset="SJ2W" device="" package3d_urn="urn:adsk.eagle:package:15474/1"/>

Commit message: Added population plan
Parts:
- L1: value 600Ohm@100 MHz -> 742792651
Changed lines of the file:
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@@
 <part name="P+5" library="supply1" library_urn="urn:adsk.eagle:library:371" deviceset="+5V" device=""/>
 <part name="GND30" library="supply1" library_urn="urn:adsk.eagle:library:371" deviceset="GND" device=""/>
-<part name="L1" library="Wurth_EMC Components_WE-CBF" library_urn="urn:adsk.eagle:library:14283147" deviceset="WE-CBF_0603" device="_HC" package3d_urn="urn:adsk.eagle:package:7784395/7" technology="_742792651" value="600Ohm@100 MHz"/>
+<part name="L1" library="Wurth_EMC Components_WE-CBF" library_urn="urn:adsk.eagle:library:14283147" deviceset="WE-CBF_0603" device="_HC" package3d_urn="urn:adsk.eagle:package:7784395/7" technology="_742792651" value="742792651"/>
 <part name="C1" library="rcl" library_urn="urn:adsk.eagle:library:334" deviceset="CPOL-EU" device="UD-4X5,8" package3d_urn="urn:adsk.eagle:package:23474/1" override_package3d_urn="urn:adsk.eagle:package:42845563/2" override_package_urn="urn:adsk.eagle:footprint:22972/1" value="10u"/>
 <part name="C2" library="rcl" library_urn="urn:adsk.eagle:library:334" deviceset="CPOL-EU" device="UD-4X5,8" package3d_urn="urn:adsk.eagle:package:23474/1" override_package3d_urn="urn:adsk.eagle:package:42845126/2" override_package_urn="urn:adsk.eagle:footprint:22972/1" value="10u"/>
